File: I2C-adc.kicad_pcb (KiCad board)
At the start: 2 copper layers, 40 x 30 mm, 13 parts, among them J1 Conn_01x10, U1 ADS1115

Commit message: update,
Parts:
- FB1, FB2: value Ferrite_Bead_Small -> MMZ2012Y152B
- moved J1 22.6 mm to (11.4, 24.3), turned to 90 degrees
- moved R2 18.3 mm to (16.5, 20.4)
- moved R3 13.3 mm to (19.1, 20.4), turned to 270 degrees
- moved FB1 4.01 mm to (11.6, 18.3), turned to 270 degrees
- moved C2 3.42 mm to (12.7, 21.6), turned to 0 degrees
- moved R1 3.30 mm to (19.1, 16.5)
- moved R4 3.09 mm to (16.6, 16.5)
- moved U1 2.26 mm to (24.6, 19.5), turned to 180 degrees
- moved FB2 1.12 mm to (13.8, 18.3)
Connections:
- FB1 pad 1: VDD -> GND
- FB2 pad 1: GND -> VDD
- J1 pad 1: /AIN3 -> Net-(C2-Pad1)
- J1 pad 10: Net-(C2-Pad1) -> /AIN2
- J1 pad 2: /AIN2 -> Net-(C2-Pad2)
- J1 pad 3: /AIN1 -> /SDA
- J1 pad 4: /AIN0 -> /SCL
- J1 pad 7: /SDA -> /AIN0
- J1 pad 8: /SCL -> /AIN1
- J1 pad 9: Net-(C2-Pad2) -> /AIN3
- R1 pad 2: Net-(R1-Pad2) -> /ALERT
- R2 pad 2: Net-(R2-Pad2) -> /SDA
- R3 pad 2: Net-(R3-Pad2) -> /SCL
- R4 pad 1: Net-(R4-Pad1) -> /ADDR
- U1 pad 1: Net-(R4-Pad1) -> /ADDR
- U1 pad 10: Net-(R3-Pad2) -> /SCL
- U1 pad 2: Net-(R1-Pad2) -> /ALERT
- U1 pad 9: Net-(R2-Pad2) -> /SDA
Routing:
- net VDD: track 64.9 -> 12.3 mm
- net /ADDR: track 0.00 -> 28.2 mm, vias 0 -> 2
- net /ALERT: track 0.00 -> 17.8 mm, vias 0 -> 2
- net /AIN2: track 5.04 -> 21.5 mm
- net GND: track 17.9 -> 6.59 mm, vias 8 -> 14
- net Net-(C2-Pad1): track 15.8 -> 5.14 mm
- net /AIN3: track 7.79 -> 17.9 mm
- net /SDA: track 0.00 -> 9.73 mm
- net Net-(R4-Pad1): track 8.72 -> 0.00 mm
- net /SCL: track 0.00 -> 7.24 mm
- net Net-(R2-Pad2): track 6.44 -> 0.00 mm
- net Net-(R1-Pad2): track 3.53 -> 0.00 mm
- net /AIN1: track 6.54 -> 10.1 mm
- net Net-(R3-Pad2): track 3.31 -> 0.00 mm
- net Net-(C2-Pad2): track 6.75 -> 5.14 mm
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